File: kicadSchematic/rough-schematic-sketch.kicad_sch (KiCad schematic)
At the start: 25 parts, among them K1 Compressor Relay, K2 Auger Relay, M1 Compressor, M2 Auger Motor, M3 Pump, M4 Fan, Q1 Pump Mosfet, Q2 UV LED Mosfet, Q3 Fan Mosfet, SW1 Reset Button, SW2 Power Switch, SW3 Bin Switch, SW4 Float High, SW5 Float Low, SW6 Bin Light Switch

Commit message: schematic touchup and warning
Parts:
- R2: value 220 -> 220Ω
Other:
- company: (none) -> https://aspy.dev
- title: (none) -> GE Opal 2 Board replacement
Changed lines of the file:
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@@
 	(generator_version "10.0")
 	(paper "A4")
+	(title_block
+		(title "GE Opal 2 Board replacement")
+		(date "2026-08-08")
+		(company "https://aspy.dev")
+		(comment 1 "https://github.com/someaspy")
+		(comment 2 "amb@aspy.dev")
+	)
 	(text "Float High is closed when the internal tank is full (Normally Open)\nFloat Low is closes when the internal tank is empty (Normally Closed)"
 		(exclude_from_sim no)
@@
 	)
 	(junction
-		(at 212.09 96.52)
-		(diameter 0)
-		(color 0 0 0 0)
-	)
-	(junction
 		(at 209.55 74.93)
 		(diameter 0)
@@
 	(wire
 		(pts
-			(xy 217.17 72.39) (xy 217.17 74.93)
-		)
-		(stroke
-			(width 0)
-			(type default)
-		)
-	)
-	(wire
-		(pts
-			(xy 212.09 106.68) (xy 212.09 96.52)
-		)
-		(stroke
-			(width 0)
-			(type default)
-		)
-	)
-	(wire
-		(pts
 			(xy 83.82 182.88) (xy 83.82 176.53)
 		)
@@
 	(wire
 		(pts
-			(xy 217.17 74.93) (xy 209.55 74.93)
+			(xy 209.55 74.93) (xy 227.33 74.93)
 		)
 		(stroke
@@
 	(wire
 		(pts
-			(xy 227.33 72.39) (xy 217.17 72.39)
-		)
-		(stroke
-			(width 0)
-			(type default)
-		)
-	)
-	(wire
-		(pts
 			(xy 115.57 82.55) (xy 115.57 86.36)
 		)
@@
 	(wire
 		(pts
-			(xy 209.55 96.52) (xy 212.09 96.52)
+			(xy 209.55 96.52) (xy 218.44 96.52)
 		)
 		(stroke
@@
 	(wire
 		(pts
-			(xy 80.01 113.03) (xy 91.44 113.03)
+			(xy 227.33 74.93) (xy 227.33 72.39)
 		)
 		(stroke
@@
 	(wire
 		(pts
-			(xy 109.22 119.38) (xy 109.22 96.52)
+			(xy 80.01 113.03) (xy 91.44 113.03)
 		)
 		(stroke
@@
 	(wire
 		(pts
-			(xy 227.33 124.46) (xy 212.09 124.46)
+			(xy 109.22 119.38) (xy 109.22 96.52)
 		)
 		(stroke
@@
 	(wire
 		(pts
-			(xy 50.8 71.12) (xy 48.26 71.12)
+			(xy 227.33 124.46) (xy 212.09 124.46)
 		)
 		(stroke
@@
 	(wire
 		(pts
-			(xy 186.69 134.62) (xy 124.46 134.62)
+			(xy 50.8 71.12) (xy 48.26 71.12)
 		)
 		(stroke
@@
 	(wire
 		(pts
-			(xy 212.09 96.52) (xy 218.44 96.52)
+			(xy 186.69 134.62) (xy 124.46 134.62)
 		)
 		(stroke
@@
 		)
 		(instances
-			(project "rough-schematic-sketch]"
+			(project "rough-schematic-sketch"
 				(path "/3caecd39-8377-4639-951b-eef5198ca2fc"
 					(reference "#PWR011")
@@
 		)
 		(instances
-			(project "rough-schematic-sketch]"
+			(project "rough-schematic-sketch"
 				(path "/3caecd39-8377-4639-951b-eef5198ca2fc"
 					(reference "MES1")
@@
 		)
 		(instances
-			(project "rough-schematic-sketch]"
+			(project "rough-schematic-sketch"
 				(path "/3caecd39-8377-4639-951b-eef5198ca2fc"
 					(reference "#PWR06")
@@
 		)
 		(instances
-			(project "rough-schematic-sketch]"
+			(project "rough-schematic-sketch"
 				(path "/3caecd39-8377-4639-951b-eef5198ca2fc"
 					(reference "D5")
@@
 		)
 		(instances
-			(project "rough-schematic-sketch]"
+			(project "rough-schematic-sketch"
 				(path "/3caecd39-8377-4639-951b-eef5198ca2fc"
 					(reference "M3")
@@
 		)
 		(instances
-			(project "rough-schematic-sketch]"
+			(project "rough-schematic-sketch"
 				(path "/3caecd39-8377-4639-951b-eef5198ca2fc"
 					(reference "#PWR08")
@@
 		)
 		(instances
-			(project "rough-schematic-sketch]"
+			(project "rough-schematic-sketch"
 				(path "/3caecd39-8377-4639-951b-eef5198ca2fc"
 					(reference "#PWR018")
@@
 		)
 		(instances
-			(project "rough-schematic-sketch]"
+			(project "rough-schematic-sketch"
 				(path "/3caecd39-8377-4639-951b-eef5198ca2fc"
 					(reference "K1")
@@
 		)
 		(instances
-			(project "rough-schematic-sketch]"
+			(project "rough-schematic-sketch"
 				(path "/3caecd39-8377-4639-951b-eef5198ca2fc"
 					(reference "#PWR020")
@@
 		)
 		(instances
-			(project "rough-schematic-sketch]"
+			(project "rough-schematic-sketch"
 				(path "/3caecd39-8377-4639-951b-eef5198ca2fc"
 					(reference "R4")
@@
 		)
 		(instances
-			(project "rough-schematic-sketch]"
+			(project "rough-schematic-sketch"
 				(path "/3caecd39-8377-4639-951b-eef5198ca2fc"
 					(reference "#PWR03")
@@
 		)
 		(instances
-			(project "rough-schematic-sketch]"
+			(project "rough-schematic-sketch"
 				(path "/3caecd39-8377-4639-951b-eef5198ca2fc"
 					(reference "#PWR017")
@@
 		)
 		(instances
-			(project "rough-schematic-sketch]"
+			(project "rough-schematic-sketch"
 				(path "/3caecd39-8377-4639-951b-eef5198ca2fc"
 					(reference "#PWR01")
@@
 		)
 		(instances
-			(project "rough-schematic-sketch]"
+			(project "rough-schematic-sketch"
 				(path "/3caecd39-8377-4639-951b-eef5198ca2fc"
 					(reference "#PWR016")
@@
 		)
 		(instances
-			(project "rough-schematic-sketch]"
+			(project "rough-schematic-sketch"
 				(path "/3caecd39-8377-4639-951b-eef5198ca2fc"
 					(reference "SW1")
@@
 		)
 		(instances
-			(project "rough-schematic-sketch]"
+			(project "rough-schematic-sketch"
 				(path "/3caecd39-8377-4639-951b-eef5198ca2fc"
 					(reference "M1")
@@
 		)
 		(instances
-			(project "rough-schematic-sketch]"
+			(project "rough-schematic-sketch"
 				(path "/3caecd39-8377-4639-951b-eef5198ca2fc"
 					(reference "Q2")
@@
 		)
 		(instances
-			(project "rough-schematic-sketch]"
+			(project "rough-schematic-sketch"
 				(path "/3caecd39-8377-4639-951b-eef5198ca2fc"
 					(reference "M4")
@@
 		)
 		(instances
-			(project "rough-schematic-sketch]"
+			(project "rough-schematic-sketch"
 				(path "/3caecd39-8377-4639-951b-eef5198ca2fc"
 					(reference "M2")
@@
 		)
 		(instances
-			(project "rough-schematic-sketch]"
+			(project "rough-schematic-sketch"
 				(path "/3caecd39-8377-4639-951b-eef5198ca2fc"
 					(reference "#PWR09")
@@
 		)
 		(instances
-			(project "rough-schematic-sketch]"
+			(project "rough-schematic-sketch"
 				(path "/3caecd39-8377-4639-951b-eef5198ca2fc"
 					(reference "#PWR04")
@@
 		)
 		(instances
-			(project "rough-schematic-sketch]"
+			(project "rough-schematic-sketch"
 				(path "/3caecd39-8377-4639-951b-eef5198ca2fc"
 					(reference "R3")
@@
 		)
 		(instances
-			(project "rough-schematic-sketch]"
+			(project "rough-schematic-sketch"
 				(path "/3caecd39-8377-4639-951b-eef5198ca2fc"
 					(reference "K2")
@@
 		)
 		(instances
-			(project "rough-schematic-sketch]"
+			(project "rough-schematic-sketch"
 				(path "/3caecd39-8377-4639-951b-eef5198ca2fc"
 					(reference "#PWR05")
@@
 		)
 		(instances
-			(project "rough-schematic-sketch]"
+			(project "rough-schematic-sketch"
 				(path "/3caecd39-8377-4639-951b-eef5198ca2fc"
 					(reference "Q3")
@@
 		)
 		(instances
-			(project "rough-schematic-sketch]"
+			(project "rough-schematic-sketch"
 				(path "/3caecd39-8377-4639-951b-eef5198ca2fc"
 					(reference "A1")
@@
 		)
 		(instances
-			(project "rough-schematic-sketch]"
+			(project "rough-schematic-sketch"
 				(path "/3caecd39-8377-4639-951b-eef5198ca2fc"
 					(reference "SW2")
@@
 		)
 		(instances
-			(project "rough-schematic-sketch]"
+			(project "rough-schematic-sketch"
 				(path "/3caecd39-8377-4639-951b-eef5198ca2fc"
 					(reference "#PWR012")
@@
 		)
 		(instances
-			(project "rough-schematic-sketch]"
+			(project "rough-schematic-sketch"
 				(path "/3caecd39-8377-4639-951b-eef5198ca2fc"
 					(reference "SW4")
@@
 		)
 		(instances
-			(project "rough-schematic-sketch]"
+			(project "rough-schematic-sketch"
 				(path "/3caecd39-8377-4639-951b-eef5198ca2fc"
 					(reference "Q1")
@@
 		)
 		(instances
-			(project "rough-schematic-sketch]"
+			(project "rough-schematic-sketch"
 				(path "/3caecd39-8377-4639-951b-eef5198ca2fc"
 					(reference "SW6")
@@
 		)
 		(instances
-			(project "rough-schematic-sketch]"
+			(project "rough-schematic-sketch"
 				(path "/3caecd39-8377-4639-951b-eef5198ca2fc"
 					(reference "D1")
@@
 		)
 		(instances
-			(project "rough-schematic-sketch]"
+			(project "rough-schematic-sketch"
 				(path "/3caecd39-8377-4639-951b-eef5198ca2fc"
 					(reference "#PWR015")
@@
 		)
 		(instances
-			(project "rough-schematic-sketch]"
+			(project "rough-schematic-sketch"
 				(path "/3caecd39-8377-4639-951b-eef5198ca2fc"
 					(reference "SW3")
@@
 		)
 		(instances
-			(project "rough-schematic-sketch]"
+			(project "rough-schematic-sketch"
 				(path "/3caecd39-8377-4639-951b-eef5198ca2fc"
 					(reference "D4")
@@
 		)
 		(instances
-			(project "rough-schematic-sketch]"
+			(project "rough-schematic-sketch"
 				(path "/3caecd39-8377-4639-951b-eef5198ca2fc"
 					(reference "#PWR010")
@@
 		)
 		(instances
-			(project "rough-schematic-sketch]"
+			(project "rough-schematic-sketch"
 				(path "/3caecd39-8377-4639-951b-eef5198ca2fc"
 					(reference "D3")
@@
 		)
 		(instances
-			(project "rough-schematic-sketch]"
+			(project "rough-schematic-sketch"
 				(path "/3caecd39-8377-4639-951b-eef5198ca2fc"
 					(reference "#PWR07")
@@
 		)
 		(instances
-			(project "rough-schematic-sketch]"
+			(project "rough-schematic-sketch"
 				(path "/3caecd39-8377-4639-951b-eef5198ca2fc"
 					(reference "#PWR019")
@@
 		)
 		(instances
-			(project "rough-schematic-sketch]"
+			(project "rough-schematic-sketch"
 				(path "/3caecd39-8377-4639-951b-eef5198ca2fc"
 					(reference "#PWR02")
@@
 		)
 		(instances
-			(project "rough-schematic-sketch]"
+			(project "rough-schematic-sketch"
 				(path "/3caecd39-8377-4639-951b-eef5198ca2fc"
 					(reference "#PWR014")
@@
 		)
 		(instances
-			(project "rough-schematic-sketch]"
+			(project "rough-schematic-sketch"
 				(path "/3caecd39-8377-4639-951b-eef5198ca2fc"
 					(reference "SW5")
@@
 		)
 		(instances
-			(project "rough-schematic-sketch]"
+			(project "rough-schematic-sketch"
 				(path "/3caecd39-8377-4639-951b-eef5198ca2fc"
 					(reference "D2")
@@
 			)
 		)
-		(property "Value" "220"
+		(property "Value" "220Ω"
 			(at 91.186 117.348 90)
 			(show_name no)
@@
 		)
 		(instances
-			(project "rough-schematic-sketch]"
+			(project "rough-schematic-sketch"
 				(path "/3caecd39-8377-4639-951b-eef5198ca2fc"
 					(reference "R2")
@@
 		)
 		(instances
-			(project "rough-schematic-sketch]"
+			(project "rough-schematic-sketch"
 				(path "/3caecd39-8377-4639-951b-eef5198ca2fc"
 					(reference "#PWR013")

Commit message: a word of warning added to schematic
Parts:
- removed A1: Arduino_Nano_v2.x, Module:Arduino_Nano, symbol MCU_Module:Arduino_Nano_v2.x
- removed SW6: Bin Light Switch, symbol Switch:SW_SPST
- added A1: Arduino_Nano_v3.x, Module:Arduino_Nano, symbol MCU_Module:Arduino_Nano_v3.x
- added R1: 100Ω, symbol Device:R_US
Connections:
- net +5V: now also A1.27 (+5V)
- net GND: now also A1.29 (GND)
- net at K1.A2: now also A1.11 (D8)
- net at R3.1, R4.1: now also A1.16 (D13)
- net at SW1.1: now also A1.28 (~{RESET})
- net at Q2.1 (G): now also A1.14 (D11)
- net at K2.A2: now also A1.12 (D9)
- net at Q3.1 (G): now also A1.13 (D10)
- net at R2.2: now also A1.10 (D7)
- net at Q1.1 (G): now also A1.15 (D12)
- net at SW2.2 (B): now also A1.5 (D2)
- net at SW3.2: now also A1.6 (D3)
- net at SW4.2 (B): now also A1.8 (D5)
- net at SW5.2 (B): now also A1.9 (D6)
- net at D1.2 (A): now also R1.1
- new net: A1.7 (D4), R1.2
Other:
- note added: "Be careful how you source 12V here!!! Say, using a buck converter your 5V powersource will backfeed from the arduino when the machine is unplugged you will probably get Welder's Flash from the light if you try to inspect it (ask me how I know)"
